Commit message: sensors commented for error correction

File: agv_low/robots/agv_urdf_youbot_collisionwheel.xacro (robot description, xacro)
@@ -34,4 +34,5 @@
   		<xacro:mecanum_wheel_visual prefix="${prefix}back_right" angle="1" wheel_pos="1" parent="${prefix}base_link" />
   		<!-- IMU -->
+<!--
 		<xacro:sensor_imu_hector prefix="$(arg prefix)imu" parent="$(arg prefix)base_link">
 			<origin xyz="0.48 0.0 0.338" rpy="0 0 0"/>
@@ -43,12 +44,13 @@
 			<origin xyz="0.060 -0.349 0.338" rpy="0 0 3.1416"/>
 		</xacro:sensor_sick_s300>
-		<xacro:sensor_asus_xtion_pro prefix="$(arg prefix)xtion" parent="$(arg prefix)base_link" >
+		<xacro:sensor_asus_xtion_pro prefix="$(arg prefix)xtion" parent="$(arg prefix)base_link" > -->
 			<!--<origin xyz="0.900 -0.0235 0.338" rpy="0 0 0" /> -->
-			<origin xyz="0.900 -0.0235 0.35075" rpy="0 1.571 -3.1416" />
+<!--			<origin xyz="0.900 -0.0235 0.35075" rpy="0 1.571 -3.1416" />
 		</xacro:sensor_asus_xtion_pro>
-		<xacro:sensor_asus_xtion_pro_stand prefix="$(arg prefix)xtion_stand" parent="$(arg prefix)base_link" >
+		<xacro:sensor_asus_xtion_pro_stand prefix="$(arg prefix)xtion_stand" parent="$(arg prefix)base_link" > -->
 			<!--<origin xyz="0.900 -0.0235 0.338" rpy="0 0 0" /> -->
-			<origin xyz="0.900 -0.0235 0.338" rpy="0 0 0" />
+<!--			<origin xyz="0.900 -0.0235 0.338" rpy="0 0 0" />
 		</xacro:sensor_asus_xtion_pro_stand>
+-->
    	</xacro:macro>
    <!-- Gazebo ros control pluggins -->
